Commit message: 4 standoff_rods added; rviz file re-calibrated

File: urdf/barista_robot_model.urdf (robot description, URDF)
Before this commit: robot barista_robot, 2 links, 1 joints
Links:
- added link standoff_rod_back_left; visual cylinder length=0.22 radius=0.01
- added link standoff_rod_back_right; visual cylinder length=0.22 radius=0.01
- added link standoff_rod_front_left; visual cylinder length=0.22 radius=0.01
- added link standoff_rod_front_right; visual cylinder length=0.22 radius=0.01
- link chassis: geometry visual cylinder length=0.155 radius=0.178
Joints:
- added joint standoff_rod_BL_to_chassis_joint: type fixed, parent chassis, child standoff_rod_back_left, origin xyz=-0.05 0.12 0.1875 rpy=0 0 0
- added joint standoff_rod_BR_to_chassis_joint: type fixed, parent chassis, child standoff_rod_back_right, origin xyz=-0.05 -0.12 0.1875 rpy=0 0 0
- added joint standoff_rod_FL_to_chassis_joint: type fixed, parent chassis, child standoff_rod_front_left, origin xyz=0.05 0.12 0.1875 rpy=0 0 0
- added joint standoff_rod_FR_to_chassis_joint: type fixed, parent chassis, child standoff_rod_front_right, origin xyz=0.05 -0.12 0.1875 rpy=0 0 0

Commit message: added cup_tray

File: urdf/barista_robot_model.urdf (robot description, URDF)
Before this commit: robot barista_robot, 6 links, 5 joints
Links:
- added link cup_tray; visual cylinder length=0.09 radius=0.178
Joints:
- added joint cup_tray_to_chassis_joint: type fixed, parent chassis, child cup_tray, origin xyz=0 0 0.3425 rpy=0 0 0

Commit message: add 2 motor wheels &2 caster wheels

File: urdf/barista_robot_model.urdf (robot description, URDF)
Before this commit: robot barista_robot, 7 links, 6 joints
Links:
- added link back_pitch_link; visual sphere radius=0.0352
- added link back_roll_link; visual cylinder length=0.005 radius=0.0352
- added link back_yaw_link; visual cylinder length=0.005 radius=0.0352
- added link front_pitch_link; visual sphere radius=0.0352
- added link front_roll_link; visual cylinder length=0.005 radius=0.0352
- added link front_yaw_link; visual cylinder length=0.005 radius=0.0352
- added link left_wheel; visual cylinder length=0.0206 radius=0.0352
- added link right_wheel; visual cylinder length=0.0206 radius=0.0352
Joints:
- added joint back_pitch_joint: type continuous, parent back_roll_link, child back_pitch_link, origin xyz=0 0 0 rpy=0 0 0, axis 0 1 0, limit effort=1000.0 velocity=100.0
- added joint back_roll_joint: type continuous, parent back_yaw_link, child back_roll_link, origin xyz=0 0 0 rpy=0 0 0, axis 1 0 0, limit effort=1000.0 velocity=100.0
- added joint back_yaw_joint: type continuous, parent chassis, child back_yaw_link, origin xyz=-0.12 0 -0.0775 rpy=0 0 0, axis 0 0 1, limit effort=1000.0 velocity=100.0
- added joint front_pitch_joint: type continuous, parent front_roll_link, child front_pitch_link, origin xyz=0 0 0 rpy=0 0 0, axis 0 1 0, limit effort=1000.0 velocity=100.0
- added joint front_roll_joint: type continuous, parent front_yaw_link, child front_roll_link, origin xyz=0 0 0 rpy=0 0 0, axis 1 0 0, limit effort=1000.0 velocity=100.0
- added joint front_yaw_joint: type continuous, parent chassis, child front_yaw_link, origin xyz=0.12 0 -0.0775 rpy=0 0 0, axis 0 0 1, limit effort=1000.0 velocity=100.0
- added joint joint_left_wheel: type continuous, parent chassis, child left_wheel, origin xyz=0 0.128 -0.0775 rpy=0 0 0, axis 0 1 0, limit effort=10000 velocity=1000
- added joint joint_right_wheel: type continuous, parent chassis, child right_wheel, origin xyz=0 -0.128 -0.0775 rpy=0 0 0, axis 0 1 0, limit effort=10000 velocity=1000

Commit message: added inertias & collision to all links

File: urdf/barista_robot_model.urdf (robot description, URDF)
Before this commit: robot barista_robot, 15 links, 14 joints
Links:
- link back_pitch_link: mass None -> 0.01; geometry collision sphere radius=0.0352; visual sphere radius=0.0352
- link back_roll_link: mass None -> 0.01; geometry collision cylinder length=0.005 radius=0.0352; visual cylinder length=0.005 radius=0.0352
- link back_yaw_link: mass None -> 0.01; geometry collision cylinder length=0.005 radius=0.0352; visual cylinder length=0.005 radius=0.0352
- link chassis: mass None -> 0.2; geometry collision cylinder length=0.155 radius=0.178; visual cylinder length=0.155 radius=0.178
- link cup_tray: mass None -> 0.05; geometry collision cylinder length=0.09 radius=0.178; visual cylinder length=0.09 radius=0.178
- link front_pitch_link: mass None -> 0.01; geometry collision sphere radius=0.0352; visual sphere radius=0.0352
- link front_roll_link: mass None -> 0.01; geometry collision cylinder length=0.005 radius=0.0352; visual cylinder length=0.005 radius=0.0352
- link front_yaw_link: mass None -> 0.01; geometry collision cylinder length=0.005 radius=0.0352; visual cylinder length=0.005 radius=0.0352
- link left_wheel: mass None -> 0.01; geometry collision cylinder length=0.0206 radius=0.0352; visual cylinder length=0.0206 radius=0.0352
- link right_wheel: mass None -> 0.01; geometry collision cylinder length=0.0206 radius=0.0352; visual cylinder length=0.0206 radius=0.0352
- link standoff_rod_back_left: mass None -> 0.02; geometry collision cylinder length=0.22 radius=0.01; visual cylinder length=0.22 radius=0.01
- link standoff_rod_back_right: mass None -> 0.02; geometry collision cylinder length=0.22 radius=0.01; visual cylinder length=0.22 radius=0.01
- link standoff_rod_front_left: mass None -> 0.02; geometry collision cylinder length=0.22 radius=0.01; visual cylinder length=0.22 radius=0.01
- link standoff_rod_front_right: mass None -> 0.02; geometry collision cylinder length=0.22 radius=0.01; visual cylinder length=0.22 radius=0.01

Commit message: laser urdf added; working in Rviz

File: urdf/barista_robot_model.urdf (robot description, URDF)
Before this commit: robot barista_robot, 15 links, 14 joints
Links:
- added link laser_scan_frame
- added link laser_scan_link, mass 0.01; collision box size=0.074986 0.074935 0.0408; visual mesh filename=package://barista_robot_description/meshes/hokuyo_urg_04lx.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 scale=1.0 1.0 1.0
Joints:
- added joint laser_scan_frame_joint: type fixed, parent laser_scan_link, child laser_scan_frame, origin xyz=0 0 0.03 rpy=0 0 0, axis 0 0 0
- added joint laser_scan_link_joint: type fixed, parent chassis, child laser_scan_link, origin xyz=0.0 0.0 0.0775 rpy=0 0 0
