Commit message: added joint_state_publisher_gui in launch; added macro for wheel

File: xacro/barista_robot_model.urdf.xacro (robot description, xacro)
@@ -1,4 +1,6 @@
 <?xml version="1.0"?>
 <robot xmlns:xacro="http://www.ros.org/wiki/xacro" name="barista_bot">
+<xacro:include filename="$(find barista_robot_description)/xacro/wheel.xacro" />
+<!-- <xacro:include filename="$(find barista_robot_description)/xacro/standoff.xacro" /> -->
 <!-- Color -->
 <material name="red">
@@ -17,7 +19,4 @@
     <color rgba="0.0 0.0 0.0 1"/>
 </material>
-<material name="white">
-    <color rgba="1.0 1.0 1.0 1"/>
-</material>
 <material name="box_bot_blue">
     <color rgba="0.088656 0.428691 0.491021 1"/>
@@ -26,6 +25,4 @@
 <xacro:property name="base_width" value="0.356"/>
 <xacro:property name="base_height" value="0.155"/>
-<xacro:property name="standoff_height" value="0.22"/>
-<xacro:property name="standoff_diameter" value="0.02"/>
 <xacro:property name="cup_tray_width" value="0.32"/>
 <xacro:property name="cup_tray_height" value="0.09"/>
@@ -59,3 +56,13 @@
 <child link="chassis" />
 </joint>
+<!-- Wheel Macro -->
+<xacro:wheel wheel_name="left_wheel"/>
+<joint name="joint_left_wheel" type="continuous">
+    <origin rpy="0 0 0" xyz="0 0.128 -0.0775"/>
+    <child link="left_wheel"/>
+    <parent link="chassis"/>
+    <axis rpy="0 0 0" xyz="0 1 0"/>
+    <limit effort="10000" velocity="1000"/>
+    <joint_properties damping="1.0" friction="1.0"/>
+</joint>
 </robot>

Commit message: 2 motor wheels added

File: xacro/barista_robot_model.urdf.xacro (robot description, xacro)
@@ -66,3 +66,13 @@
     <joint_properties damping="1.0" friction="1.0"/>
 </joint>
+<xacro:wheel wheel_name="right_wheel"/>
+<joint name="joint_right_wheel" type="continuous">
+    <origin rpy="0 0 0" xyz="0 -0.128 -0.0775"/>
+    <child link="right_wheel"/>
+    <parent link="chassis"/>
+    <axis rpy="0 0 0" xyz="0 1 0"/>
+    <limit effort="10000" velocity="1000"/>
+    <joint_properties damping="1.0" friction="1.0"/>
+</joint>
+<!--  -->
 </robot>

Commit message: 4 standoffs added

File: xacro/barista_robot_model.urdf.xacro (robot description, xacro)
@@ -2,5 +2,5 @@
 <robot xmlns:xacro="http://www.ros.org/wiki/xacro" name="barista_bot">
 <xacro:include filename="$(find barista_robot_description)/xacro/wheel.xacro" />
-<!-- <xacro:include filename="$(find barista_robot_description)/xacro/standoff.xacro" /> -->
+<xacro:include filename="$(find barista_robot_description)/xacro/standoff.xacro" />
 <!-- Color -->
 <material name="red">
@@ -75,4 +75,28 @@
     <joint_properties damping="1.0" friction="1.0"/>
 </joint>
-<!--  -->
+<!-- Standoff -->
+<xacro:standoff standoff_name="standoff_rod_front_left"/>
+<joint name="standoff_rod_FL_to_chassis_joint" type="fixed">
+    <origin rpy="0 0 0" xyz="0.05 0.12 0.1875" />
+    <parent link="chassis" />
+    <child link="standoff_rod_front_left" />
+</joint>
+<xacro:standoff standoff_name="standoff_rod_back_left"/>
+<joint name="standoff_rod_BL_to_chassis_joint" type="fixed">
+    <origin rpy="0 0 0" xyz="-0.05 0.12 0.1875" />
+    <parent link="chassis" />
+    <child link="standoff_rod_back_left" />
+</joint>
+<xacro:standoff standoff_name="standoff_rod_front_right"/>
+<joint name="standoff_rod_FR_to_chassis_joint" type="fixed">
+    <origin rpy="0 0 0" xyz="0.05 -0.12 0.1875" />
+    <parent link="chassis" />
+    <child link="standoff_rod_front_right" />
+</joint>
+<xacro:standoff standoff_name="standoff_rod_back_right"/>
+<joint name="standoff_rod_BR_to_chassis_joint" type="fixed">
+    <origin rpy="0 0 0" xyz="-0.05 -0.12 0.1875" />
+    <parent link="chassis" />
+    <child link="standoff_rod_back_right" />
+</joint>
 </robot>

Commit message: cup_holder added

File: xacro/barista_robot_model.urdf.xacro (robot description, xacro)
@@ -52,7 +52,7 @@
 </link>
 <joint name="base_link_joint" type="fixed">
-<origin rpy="0 0 0" xyz="0 0 0" />
-<parent link="base_link" />
-<child link="chassis" />
+    <origin rpy="0 0 0" xyz="0 0 0" />
+    <parent link="base_link" />
+    <child link="chassis" />
 </joint>
 <!-- Wheel Macro -->
@@ -100,3 +100,11 @@
     <child link="standoff_rod_back_right" />
 </joint>
+<!-- Cup Tray -->
+<xacro:cup_holder cup_holder_name="cup_tray"/>
+<joint name="cup_tray_to_chassis_joint" type="fixed">
+    <origin rpy="0 0 0" xyz="0 0 0.3425" />
+    <parent link="chassis" />
+    <child link="cup_tray" />
+</joint>
+<!-- Caster Wheels -->
 </robot>

Commit message: fixed cup_holder include tag; dup in color definition

File: xacro/barista_robot_model.urdf.xacro (robot description, xacro)
@@ -3,4 +3,5 @@
 <xacro:include filename="$(find barista_robot_description)/xacro/wheel.xacro" />
 <xacro:include filename="$(find barista_robot_description)/xacro/standoff.xacro" />
+<xacro:include filename="$(find barista_robot_description)/xacro/cup_holder_tray.xacro" />
 <!-- Color -->
 <material name="red">

File: xacro/cup_holder_tray.xacro (robot description, xacro)
@@ -1,8 +1,4 @@
 <?xml version="1.0"?>
 <robot xmlns:xacro="http://www.ros.org/wiki/xacro">
-<!-- RVIZ Color -->
-<material name="blue">
-    <color rgba="0.0 0.0 1.0 1"/>
-</material>
 <!-- Parameters -->
 <xacro:property name="cup_holder_height" value="0.09"/>

Commit message: added laser; incomplete gazebo setup

File: xacro/barista_robot_model.urdf.xacro (robot description, xacro)
@@ -109,3 +109,280 @@
 </joint>
 <!-- Caster Wheels -->
+   <!-- yaw -->
+  <link name="front_yaw_link">
+    <visual>
+        <origin rpy="0 1.5707 1.5707" xyz="0 0 0"/>
+        <geometry>
+          <cylinder length="0.005" radius="0.0352"/>
+        </geometry>
+        <material name="blue"/>
+    </visual>
+    <inertial>
+      <mass value="0.01"/>
+      <origin rpy="0 0 0" xyz="0 0 0"/>
+      <inertia ixx="0.0000031184" ixy="0" ixz="0" iyy="0.0000031184" iyz="0" izz="0.000006195"/>
+    </inertial>
+    <collision>
+        <origin rpy="0 1.5707 1.5707" xyz="0 0 0"/>
+        <geometry>
+          <cylinder length="0.005" radius="0.0352"/>
+        </geometry>
+    </collision>
+  </link>
+    <gazebo reference="front_yaw_link">
+    <kp>1000000000000000000000000000.0</kp>
+    <kd>1000000000000000000000000000.0</kd>
+    <mu1>0.1</mu1>
+    <mu2>0.1</mu2>
+  </gazebo>
+  <joint name="front_yaw_joint" type="continuous">
+    <origin rpy="0 0 0" xyz="0.12 0 -0.0775" />
+    <parent link="chassis" />
+    <child link="front_yaw_link" />
+    <axis xyz="0 0 1" />
+    <limit effort="1000.0" velocity="100.0" />
+    <dynamics damping="0.0" friction="0.1"/>
+  </joint>
+<!-- roll -->
+  <link name="front_roll_link">
+      <visual>
+        <origin rpy="0 1.5707 1.5707" xyz="0 0 0"/>
+        <geometry>
+          <cylinder length="0.005" radius="0.0352"/>
+        </geometry>
+        <material name="red"/>
+      </visual>
+    <inertial>
+      <mass value="0.01"/>
+      <origin rpy="0 0 0" xyz="0 0 0"/>
+      <inertia ixx="0.0000031184" ixy="0" ixz="0" iyy="0.0000031184" iyz="0" izz="0.000006195"/>
+    </inertial>
+    <collision>
+        <origin rpy="0 1.5707 1.5707" xyz="0 0 0"/>
+        <geometry>
+          <cylinder length="0.005" radius="0.0352"/>
+        </geometry>
+    </collision>
+  </link>
+    <gazebo reference="front_roll_link">
+    <kp>1000000000000000000000000000.0</kp>
+    <kd>1000000000000000000000000000.0</kd>
+    <mu1>0.1</mu1>
+    <mu2>0.1</mu2>
+  </gazebo>
+  <joint name="front_roll_joint" type="continuous">
+    <origin rpy="0 0 0" xyz="0 0 0" />
+    <parent link="front_yaw_link" />
+    <child link="front_roll_link" />
+    <axis xyz="1 0 0" />
+    <limit effort="1000.0" velocity="100.0" />
+    <dynamics damping="0.0" friction="0.1"/>
+  </joint>
+<!-- pitch -->
+  <link name="front_pitch_link">
+    <visual>
+      <origin rpy="0 1.5707 1.5707" xyz="0 0 0"/>
+      <geometry>
+        <sphere radius="0.0352"/>
+      </geometry>
+      <material name="green_dark"/>
+    </visual>
+    <inertial>
+      <mass value="0.01"/>
+      <origin rpy="0 0 0" xyz="0 0 0"/>
+      <inertia ixx="0.00000826" ixy="0" ixz="0" iyy="00.00000826" iyz="0" izz="0.00000826"/>
+    </inertial>
+    <collision>
+      <origin rpy="0 1.5707 1.5707" xyz="0 0 0"/>
+      <geometry>
+        <sphere radius="0.0352"/>
+      </geometry>
+    </collision>
+  </link>
+    <gazebo reference="front_pitch_link">
+    <kp>1000000000000000000000000000.0</kp>
+    <kd>1000000000000000000000000000.0</kd>
+    <mu1>0.1</mu1>
+    <mu2>0.1</mu2>
+    <material>Gazebo/Purple</material>
+  </gazebo>
+  <joint name="front_pitch_joint" type="continuous">
+    <origin rpy="0 0 0" xyz="0 0 0" />
+    <parent link="front_roll_link" />
+    <child link="front_pitch_link" />
+    <axis xyz="0 1 0" />
+    <limit effort="1000.0" velocity="100.0" />
+    <dynamics damping="0.0" friction="0.1"/>
+  </joint>
+<!-- Caster Wheel Back -->
+  <link name="back_yaw_link">
+    <visual>
+        <origin rpy="0 1.5707 1.5707" xyz="0 0 0"/>
+        <geometry>
+          <cylinder length="0.005" radius="0.0352"/>
+        </geometry>
+        <material name="blue"/>
+      </visual>
+    <inertial>
+      <mass value="0.01"/>
+      <origin rpy="0 0 0" xyz="0 0 0"/>
+      <inertia ixx="0.0000031184" ixy="0" ixz="0" iyy="0.0000031184" iyz="0" izz="0.000006195"/>
+    </inertial>
+    <collision>
+        <origin rpy="0 1.5707 1.5707" xyz="0 0 0"/>
+        <geometry>
+          <cylinder length="0.005" radius="0.0352"/>
+        </geometry>
+    </collision>
+  </link>
+    <gazebo reference="back_yaw_link">
+    <kp>1000000000000000000000000000.0</kp>
+    <kd>1000000000000000000000000000.0</kd>
+    <mu1>0.1</mu1>
+    <mu2>0.1</mu2>
+  </gazebo>
+  <joint name="back_yaw_joint" type="continuous">
+    <origin rpy="0 0 0" xyz="-0.12 0 -0.0775" />
+    <parent link="chassis" />
+    <child link="back_yaw_link" />
+    <axis xyz="0 0 1" />
+    <limit effort="1000.0" velocity="100.0" />
+    <dynamics damping="0.0" friction="0.1"/>
+  </joint>
+  <link name="back_roll_link">
+      <visual>
+        <origin rpy="0 1.5707 1.5707" xyz="0 0 0"/>
+        <geometry>
+          <cylinder length="0.005" radius="0.0352"/>
+        </geometry>
+        <material name="red"/>
+      </visual>
+    <inertial>
+      <mass value="0.01"/>
+      <origin rpy="0 0 0" xyz="0 0 0"/>
+      <inertia ixx="0.0000031184" ixy="0" ixz="0" iyy="0.0000031184" iyz="0" izz="0.000006195"/>
+    </inertial>
+    <collision>
+        <origin rpy="0 1.5707 1.5707" xyz="0 0 0"/>
+        <geometry>
+          <cylinder length="0.005" radius="0.0352"/>
+        </geometry>
+    </collision>
+  </link>
+  <gazebo reference="back_roll_link">
+    <kp>1000000000000000000000000000.0</kp>
+    <kd>1000000000000000000000000000.0</kd>
+    <mu1>0.1</mu1>
+    <mu2>0.1</mu2>
+  </gazebo>
+  <joint name="back_roll_joint" type="continuous">
+    <origin rpy="0 0 0" xyz="0 0 0" />
+    <parent link="back_yaw_link" />
+    <child link="back_roll_link" />
+    <axis xyz="1 0 0" />
+    <limit effort="1000.0" velocity="100.0" />
+    <dynamics damping="0.0" friction="0.1"/>
+  </joint>
+  <link name="back_pitch_link">
+    <visual>
+      <origin rpy="0 1.5707 1.5707" xyz="0 0 0"/>
+      <geometry>
+        <sphere radius="0.0352"/>
+      </geometry>
+      <material name="green_light"/>
+    </visual>
+    <inertial>
+      <mass value="0.01"/>
+      <origin rpy="0 0 0" xyz="0 0 0"/>
+      <inertia ixx="0.00000826" ixy="0" ixz="0" iyy="00.00000826" iyz="0" izz="0.00000826"/>
+    </inertial>
+    <collision>
+      <origin rpy="0 1.5707 1.5707" xyz="0 0 0"/>
+      <geometry>
+        <sphere radius="0.0352"/>
+      </geometry>
+    </collision>
+  </link>
+  <gazebo reference="back_pitch_link">
+    <kp>1000000000000000000000000000.0</kp>
+    <kd>1000000000000000000000000000.0</kd>
+    <mu1>0.1</mu1>
+    <mu2>0.1</mu2>
+    <material>Gazebo/Yellow</material>
+  </gazebo>
+  <joint name="back_pitch_joint" type="continuous">
+    <origin rpy="0 0 0" xyz="0 0 0" />
+    <parent link="back_roll_link" />
+    <child link="back_pitch_link" />
+    <axis xyz="0 1 0" />
+    <limit effort="1000.0" velocity="100.0" />
+    <dynamics damping="0.0" friction="0.1"/>
+  </joint>
+<!-- Laser -->
+<xacro:arg name="include_laser" default="true"/>
+<xacro:if value="$(arg include_laser)">
+    <!-- Laser Link -->
+    <link name="laser_scan_link">
+        <visual>
+        <origin rpy="0 0 0" xyz="0 0 0"/>
+        <geometry>
+            <mesh filename="package://barista_robot_description/meshes/hokuyo_urg_04lx.dae" scale="1.0 1.0 1.0"/>
+        </geometry>
+        </visual>
+        <collision>
+        <origin rpy="0 0 0" xyz="0 0 0.0204"/>
+        <geometry>
+            <box size="0.074986 0.074935 0.0408"/>
+        </geometry>
+        </collision>
+        <inertial>
+        <mass value="0.01"/>
+        <origin rpy="0 0 0" xyz="0 0 0.0204"/>
+        <inertia ixx="6.066578520833334e-06" ixy="0" ixz="0" iyy="6.072950163333333e-06" iyz="0" izz="9.365128684166666e-06"/>
+        </inertial>
+    </link>
+    <joint name="laser_scan_link_joint" type="fixed">
+        <origin rpy="0 0 0" xyz="0.0 0.0 0.0775"/>
+        <parent link="chassis"/>
+        <child link="laser_scan_link"/>
+    </joint>
+    <link name="laser_scan_frame">
+    </link>
+    <joint name="laser_scan_frame_joint" type="fixed">
+        <origin rpy="0 0 0" xyz="0 0 0.03"/>
+        <parent link="laser_scan_link"/>
+        <child link="laser_scan_frame"/>
+        <axis xyz="0 0 0"/>
+    </joint>
+<!-- Laser -->
+<gazebo reference="laser_scan_frame">
+    <sensor name="sensor_ray" type="ray">
+        <pose>0 0 0 0 0 0</pose>
+        <ray>
+          <scan>
+            <horizontal>
+              <samples>200</samples>
+              <resolution>1.0</resolution>
+              <min_angle>-3.14</min_angle>
+              <max_angle>3.14</max_angle>
+            </horizontal>
+          </scan>
+          <range>
+            <min>0.1</min>
+            <max>5.0</max>
+          </range>
+        </ray>
+        <always_on>true</always_on>
+        <visualize>true</visualize>
+        <update_rate>100.0</update_rate>
+        <plugin name="laser" filename="libgazebo_ros_ray_sensor.so">
+          <ros>
+            <namespace>/barista_bot</namespace>
+            <remapping>~/out:=laser_scan</remapping>
+          </ros>
+          <output_type>sensor_msgs/LaserScan</output_type>
+        </plugin>
+    </sensor>
+</gazebo>
+</xacro:if>
 </robot>

Commit message: gazebo property filled: bug discovered stuttering movement

File: xacro/barista_robot_model.urdf.xacro (robot description, xacro)
@@ -130,10 +130,4 @@
     </collision>
   </link>
-    <gazebo reference="front_yaw_link">
-    <kp>1000000000000000000000000000.0</kp>
-    <kd>1000000000000000000000000000.0</kd>
-    <mu1>0.1</mu1>
-    <mu2>0.1</mu2>
-  </gazebo>
   <joint name="front_yaw_joint" type="continuous">
     <origin rpy="0 0 0" xyz="0.12 0 -0.0775" />
@@ -165,10 +159,4 @@
     </collision>
   </link>
-    <gazebo reference="front_roll_link">
-    <kp>1000000000000000000000000000.0</kp>
-    <kd>1000000000000000000000000000.0</kd>
-    <mu1>0.1</mu1>
-    <mu2>0.1</mu2>
-  </gazebo>
   <joint name="front_roll_joint" type="continuous">
     <origin rpy="0 0 0" xyz="0 0 0" />
@@ -200,11 +188,4 @@
     </collision>
   </link>
-    <gazebo reference="front_pitch_link">
-    <kp>1000000000000000000000000000.0</kp>
-    <kd>1000000000000000000000000000.0</kd>
-    <mu1>0.1</mu1>
-    <mu2>0.1</mu2>
-    <material>Gazebo/Purple</material>
-  </gazebo>
   <joint name="front_pitch_joint" type="continuous">
     <origin rpy="0 0 0" xyz="0 0 0" />
@@ -236,10 +217,4 @@
     </collision>
   </link>
-    <gazebo reference="back_yaw_link">
-    <kp>1000000000000000000000000000.0</kp>
-    <kd>1000000000000000000000000000.0</kd>
-    <mu1>0.1</mu1>
-    <mu2>0.1</mu2>
-  </gazebo>
   <joint name="back_yaw_joint" type="continuous">
     <origin rpy="0 0 0" xyz="-0.12 0 -0.0775" />
@@ -270,10 +245,4 @@
     </collision>
   </link>
-  <gazebo reference="back_roll_link">
-    <kp>1000000000000000000000000000.0</kp>
-    <kd>1000000000000000000000000000.0</kd>
-    <mu1>0.1</mu1>
-    <mu2>0.1</mu2>
-  </gazebo>
   <joint name="back_roll_joint" type="continuous">
     <origin rpy="0 0 0" xyz="0 0 0" />
@@ -304,11 +273,4 @@
     </collision>
   </link>
-  <gazebo reference="back_pitch_link">
-    <kp>1000000000000000000000000000.0</kp>
-    <kd>1000000000000000000000000000.0</kd>
-    <mu1>0.1</mu1>
-    <mu2>0.1</mu2>
-    <material>Gazebo/Yellow</material>
-  </gazebo>
   <joint name="back_pitch_joint" type="continuous">
     <origin rpy="0 0 0" xyz="0 0 0" />
@@ -386,3 +348,118 @@
 </gazebo>
 </xacro:if>
+<!-- Gazebo Elements -->
+  <!-- Coloring Links within Gazebo  -->
+  <gazebo reference="chassis">
+    <material>Gazebo/Blue</material>
+    </gazebo>
+    <gazebo reference="cup_tray">
+        <material>Gazebo/Blue</material>
+    </gazebo>
+    <gazebo reference="standoff_rod_front_left">
+        <material>Gazebo/White</material>
+    </gazebo>
+    <gazebo reference="standoff_rod_front_right">
+        <material>Gazebo/White</material>
+    </gazebo>
+    <gazebo reference="standoff_rod_back_left">
+        <material>Gazebo/White</material>
+    </gazebo>
+    <gazebo reference="standoff_rod_back_right">
+        <material>Gazebo/White</material>
+    </gazebo>
+    <gazebo reference="back_yaw_link">
+        <material>Gazebo/Blue</material>
+    </gazebo>
+    <gazebo reference="back_roll_link">
+        <material>Gazebo/Red</material>
+    </gazebo>
+    <gazebo reference="left_wheel">
+    <kp>1000000000000000000000000000.0</kp>
+    <kd>1000000000000000000000000000.0</kd>
+    <mu1>10.0</mu1>
+    <mu2>10.0</mu2>
+    <material>Gazebo/Green</material>
+  </gazebo>
+    <gazebo reference="right_wheel">
+    <kp>1000000000000000000000000000.0</kp>
+    <kd>1000000000000000000000000000.0</kd>
+    <mu1>10.0</mu1>
+    <mu2>10.0</mu2>
+    <material>Gazebo/Orange</material>
+  </gazebo>
+    <gazebo reference="front_yaw_link">
+    <kp>1000000000000000000000000000.0</kp>
+    <kd>1000000000000000000000000000.0</kd>
+    <mu1>0.1</mu1>
+    <mu2>0.1</mu2>
+  </gazebo>
+    <gazebo reference="front_roll_link">
+    <kp>1000000000000000000000000000.0</kp>
+    <kd>1000000000000000000000000000.0</kd>
+    <mu1>0.1</mu1>
+    <mu2>0.1</mu2>
+  </gazebo>
+    <gazebo reference="front_pitch_link">
+    <kp>1000000000000000000000000000.0</kp>
+    <kd>1000000000000000000000000000.0</kd>
+    <mu1>0.1</mu1>
+    <mu2>0.1</mu2>
+    <material>Gazebo/Purple</material>
+  </gazebo>
+    <gazebo reference="back_yaw_link">
+    <kp>1000000000000000000000000000.0</kp>
+    <kd>1000000000000000000000000000.0</kd>
+    <mu1>0.1</mu1>
+    <mu2>0.1</mu2>
+  </gazebo>
+  <gazebo reference="back_roll_link">
+    <kp>1000000000000000000000000000.0</kp>
+    <kd>1000000000000000000000000000.0</kd>
+    <mu1>0.1</mu1>
+    <mu2>0.1</mu2>
+  </gazebo>
+      <gazebo reference="back_pitch_link">
+    <kp>1000000000000000000000000000.0</kp>
+    <kd>1000000000000000000000000000.0</kd>
+    <mu1>0.1</mu1>
+    <mu2>0.1</mu2>
+    <material>Gazebo/Yellow</material>
+  </gazebo>
+    <!-- Plug-ins-->
+    <!-- JOINT PUBLISHER -->
+    <gazebo>
+        <plugin name="box_bot_joint_state" filename="libgazebo_ros_joint_state_publisher.so">
+        <ros>
+            <remapping>~/out:=joint_states</remapping>
+        </ros>
+        <update_rate>30</update_rate>
+        <joint_name>joint_left_wheel</joint_name>
+        <joint_name>joint_right_wheel</joint_name>
+        <joint_name>front_yaw_joint</joint_name>
+        <joint_name>back_yaw_joint</joint_name>
+        <joint_name>front_roll_joint</joint_name>
+        <joint_name>back_roll_joint</joint_name>
+        <joint_name>front_pitch_joint</joint_name>
+        <joint_name>back_pitch_joint</joint_name>
+        </plugin>
+    </gazebo>
+    <!-- Differential drive -->
+  <gazebo>
+    <plugin filename="libgazebo_ros_diff_drive.so" name="differential_drive_controller">
+      <!-- wheels -->
+      <left_joint>joint_left_wheel</left_joint>
+      <right_joint>joint_right_wheel</right_joint>
+      <!-- kinematics -->
+      <wheel_separation>0.1</wheel_separation>
+      <wheel_diameter>0.07</wheel_diameter>
+      <!-- limits -->
+      <max_wheel_torque>1.0</max_wheel_torque>
+      <max_wheel_acceleration>2.0</max_wheel_acceleration>
+      <!-- output -->
+      <publish_odom>true</publish_odom>
+      <publish_odom_tf>true</publish_odom_tf>
+      <odometry_frame>odom</odometry_frame>
+      <robot_base_frame>base_link</robot_base_frame>
+    </plugin>
+  </gazebo>
 </robot>

Commit message: stuttering fixed: solution:'moved wheel xacro:property within macro definition'

File: xacro/barista_robot_model.urdf.xacro (robot description, xacro)
@@ -114,5 +114,5 @@
         <origin rpy="0 1.5707 1.5707" xyz="0 0 0"/>
         <geometry>
-          <cylinder length="0.005" radius="0.0352"/>
+          <cylinder length="0.005" radius="0.0352 "/>
         </geometry>
         <material name="blue"/>
@@ -429,5 +429,5 @@
     <!-- JOINT PUBLISHER -->
     <gazebo>
-        <plugin name="box_bot_joint_state" filename="libgazebo_ros_joint_state_publisher.so">
+        <plugin name="barista_bot_joint_state" filename="libgazebo_ros_joint_state_publisher.so">
         <ros>
             <remapping>~/out:=joint_states</remapping>

File: xacro/wheel.xacro (robot description, xacro)
@@ -1,7 +1,7 @@
 <?xml version="1.0"?>
 <robot xmlns:xacro="http://www.ros.org/wiki/xacro">
-<xacro:property name="wheel_width" value="0.0206"/>
-<xacro:property name="wheel_radius" value="0.0352"/>
 <xacro:macro name="wheel" params="wheel_name">
+    <xacro:property name="wheel_width" value="0.0206"/>
+    <xacro:property name="wheel_radius" value="0.0352"/>
     <link name="${wheel_name}">
         <visual>
