Commit message: added two robots launch

File: xacro/barista_robot_model.urdf.xacro (robot description, xacro)
@@ -1,4 +1,7 @@
 <?xml version="1.0"?>
 <robot xmlns:xacro="http://www.ros.org/wiki/xacro" name="barista_bot">
+<!-- Setting Robot_name -->
+<xacro:property name="robot_name" value="$(arg robot_name)"/>
+<!-- Find Parts Xacro -->
 <xacro:include filename="$(find barista_robot_description)/xacro/wheel.xacro" />
 <xacro:include filename="$(find barista_robot_description)/xacro/standoff.xacro" />
@@ -340,5 +343,5 @@
         <plugin name="laser" filename="libgazebo_ros_ray_sensor.so">
           <ros>
-            <namespace>/barista_bot</namespace>
+            <namespace>/${robot_name}</namespace>
             <remapping>~/out:=laser_scan</remapping>
           </ros>
@@ -431,4 +434,5 @@
         <plugin name="barista_bot_joint_state" filename="libgazebo_ros_joint_state_publisher.so">
         <ros>
+            <namespace>/${robot_name}</namespace>
             <remapping>~/out:=joint_states</remapping>
         </ros>
@@ -445,20 +449,26 @@
     </gazebo>
     <!-- Differential drive -->
-  <gazebo>
+ <gazebo>
     <plugin filename="libgazebo_ros_diff_drive.so" name="differential_drive_controller">
-      <!-- wheels -->
-      <left_joint>joint_left_wheel</left_joint>
-      <right_joint>joint_right_wheel</right_joint>
-      <!-- kinematics -->
-      <wheel_separation>0.1</wheel_separation>
-      <wheel_diameter>0.07</wheel_diameter>
-      <!-- limits -->
-      <max_wheel_torque>1.0</max_wheel_torque>
-      <max_wheel_acceleration>2.0</max_wheel_acceleration>
-      <!-- output -->
-      <publish_odom>true</publish_odom>
-      <publish_odom_tf>true</publish_odom_tf>
-      <odometry_frame>odom</odometry_frame>
-      <robot_base_frame>base_link</robot_base_frame>
+        <ros>
+            <namespace>/${robot_name}</namespace>
+            <remapping>/cmd_vel:=cmd_vel</remapping>
+        </ros>
+        <update_rate>100</update_rate>
+        <!-- Wheel joints -->
+        <left_joint>joint_left_wheel</left_joint>
+        <right_joint>joint_right_wheel</right_joint>
+        <!-- Kinematics -->
+        <wheel_separation>0.1</wheel_separation>
+        <wheel_diameter>0.07</wheel_diameter>
+        <publish_odom>true</publish_odom>
+        <!-- TF frames -->
+        <odometry_frame>${robot_name}/odom</odometry_frame>>
+        <robot_base_frame>${robot_name}/base_link</robot_base_frame>
+        <publish_odom_tf>true</publish_odom_tf>
+        <publish_wheel_tf>false</publish_wheel_tf>
+        <!-- Limits -->
+        <max_wheel_torque>1.0</max_wheel_torque>
+        <max_wheel_acceleration>2.0</max_wheel_acceleration>
     </plugin>
   </gazebo>

Commit message: added coloring based on robot name: 'red' if robot_name is 'rick'

File: xacro/barista_robot_model.urdf.xacro (robot description, xacro)
@@ -26,4 +26,14 @@
     <color rgba="0.088656 0.428691 0.491021 1"/>
 </material>
+<!-- Special Color for Rick -->
+<xacro:if value="${robot_name == 'rick'}">
+    <xacro:property name="gazebo_body_color" value="Gazebo/Red"/>
+    <xacro:property name="rviz_body_color" value="red"/>
+</xacro:if>
+<!-- Setting Default Color (Morty) -->
+<xacro:unless value="${robot_name == 'rick'}">
+    <xacro:property name="gazebo_body_color" value="Gazebo/Blue"/>
+    <xacro:property name="rviz_body_color" value="blue"/>
+</xacro:unless>
 <!-- Dimension Parameters -->
 <xacro:property name="base_width" value="0.356"/>
@@ -42,5 +52,5 @@
     <cylinder length="${base_height}" radius="${base_width/2}"/>
     </geometry>
-    <material name="blue"/>
+    <material name="${rviz_body_color}"/>
 </visual>
 <inertial>
@@ -105,5 +115,5 @@
 </joint>
 <!-- Cup Tray -->
-<xacro:cup_holder cup_holder_name="cup_tray"/>
+<xacro:cup_holder cup_holder_name="cup_tray" rviz_material="${rviz_body_color}"/>
 <joint name="cup_tray_to_chassis_joint" type="fixed">
     <origin rpy="0 0 0" xyz="0 0 0.3425" />
@@ -352,85 +362,85 @@
 </xacro:if>
 <!-- Gazebo Elements -->
-  <!-- Coloring Links within Gazebo  -->
-  <gazebo reference="chassis">
+<!-- Coloring Links within Gazebo  -->
+<gazebo reference="chassis">
+    <material>${gazebo_body_color}</material>
+</gazebo>
+<gazebo reference="cup_tray">
+    <material>${gazebo_body_color}</material>
+</gazebo>
+<gazebo reference="standoff_rod_front_left">
+    <material>Gazebo/White</material>
+</gazebo>
+<gazebo reference="standoff_rod_front_right">
+    <material>Gazebo/White</material>
+</gazebo>
+<gazebo reference="standoff_rod_back_left">
+    <material>Gazebo/White</material>
+</gazebo>
+<gazebo reference="standoff_rod_back_right">
+    <material>Gazebo/White</material>
+</gazebo>
+<gazebo reference="back_yaw_link">
     <material>Gazebo/Blue</material>
-    </gazebo>
-    <gazebo reference="cup_tray">
-        <material>Gazebo/Blue</material>
-    </gazebo>
-    <gazebo reference="standoff_rod_front_left">
-        <material>Gazebo/White</material>
-    </gazebo>
-    <gazebo reference="standoff_rod_front_right">
-        <material>Gazebo/White</material>
-    </gazebo>
-    <gazebo reference="standoff_rod_back_left">
-        <material>Gazebo/White</material>
-    </gazebo>
-    <gazebo reference="standoff_rod_back_right">
-        <material>Gazebo/White</material>
-    </gazebo>
-    <gazebo reference="back_yaw_link">
-        <material>Gazebo/Blue</material>
-    </gazebo>
-    <gazebo reference="back_roll_link">
-        <material>Gazebo/Red</material>
-    </gazebo>
-    <gazebo reference="left_wheel">
-    <kp>1000000000000000000000000000.0</kp>
-    <kd>1000000000000000000000000000.0</kd>
-    <mu1>10.0</mu1>
-    <mu2>10.0</mu2>
-    <material>Gazebo/Green</material>
-  </gazebo>
-    <gazebo reference="right_wheel">
-    <kp>1000000000000000000000000000.0</kp>
-    <kd>1000000000000000000000000000.0</kd>
-    <mu1>10.0</mu1>
-    <mu2>10.0</mu2>
-    <material>Gazebo/Orange</material>
-  </gazebo>
-    <gazebo reference="front_yaw_link">
-    <kp>1000000000000000000000000000.0</kp>
-    <kd>1000000000000000000000000000.0</kd>
-    <mu1>0.1</mu1>
-    <mu2>0.1</mu2>
-  </gazebo>
-    <gazebo reference="front_roll_link">
-    <kp>1000000000000000000000000000.0</kp>
-    <kd>1000000000000000000000000000.0</kd>
-    <mu1>0.1</mu1>
-    <mu2>0.1</mu2>
-  </gazebo>
-    <gazebo reference="front_pitch_link">
-    <kp>1000000000000000000000000000.0</kp>
-    <kd>1000000000000000000000000000.0</kd>
-    <mu1>0.1</mu1>
-    <mu2>0.1</mu2>
-    <material>Gazebo/Purple</material>
-  </gazebo>
-    <gazebo reference="back_yaw_link">
-    <kp>1000000000000000000000000000.0</kp>
-    <kd>1000000000000000000000000000.0</kd>
-    <mu1>0.1</mu1>
-    <mu2>0.1</mu2>
-  </gazebo>
-  <gazebo reference="back_roll_link">
-    <kp>1000000000000000000000000000.0</kp>
-    <kd>1000000000000000000000000000.0</kd>
-    <mu1>0.1</mu1>
-    <mu2>0.1</mu2>
-  </gazebo>
-      <gazebo reference="back_pitch_link">
-    <kp>1000000000000000000000000000.0</kp>
-    <kd>1000000000000000000000000000.0</kd>
-    <mu1>0.1</mu1>
-    <mu2>0.1</mu2>
-    <material>Gazebo/Yellow</material>
-  </gazebo>
+</gazebo>
+<gazebo reference="back_roll_link">
+    <material>Gazebo/Red</material>
+</gazebo>
+<gazebo reference="left_wheel">
+<kp>1000000000000000000000000000.0</kp>
+<kd>1000000000000000000000000000.0</kd>
+<mu1>10.0</mu1>
+<mu2>10.0</mu2>
+<material>Gazebo/Green</material>
+</gazebo>
+<gazebo reference="right_wheel">
+<kp>1000000000000000000000000000.0</kp>
+<kd>1000000000000000000000000000.0</kd>
+<mu1>10.0</mu1>
+<mu2>10.0</mu2>
+<material>Gazebo/Orange</material>
+</gazebo>
+<gazebo reference="front_yaw_link">
+<kp>1000000000000000000000000000.0</kp>
+<kd>1000000000000000000000000000.0</kd>
+<mu1>0.1</mu1>
+<mu2>0.1</mu2>
+</gazebo>
+<gazebo reference="front_roll_link">
+<kp>1000000000000000000000000000.0</kp>
+<kd>1000000000000000000000000000.0</kd>
+<mu1>0.1</mu1>
+<mu2>0.1</mu2>
+</gazebo>
+<gazebo reference="front_pitch_link">
+<kp>1000000000000000000000000000.0</kp>
+<kd>1000000000000000000000000000.0</kd>
+<mu1>0.1</mu1>
+<mu2>0.1</mu2>
+<material>Gazebo/Purple</material>
+</gazebo>
+<gazebo reference="back_yaw_link">
+<kp>1000000000000000000000000000.0</kp>
+<kd>1000000000000000000000000000.0</kd>
+<mu1>0.1</mu1>
+<mu2>0.1</mu2>
+</gazebo>
+<gazebo reference="back_roll_link">
+<kp>1000000000000000000000000000.0</kp>
+<kd>1000000000000000000000000000.0</kd>
+<mu1>0.1</mu1>
+<mu2>0.1</mu2>
+</gazebo>
+    <gazebo reference="back_pitch_link">
+<kp>1000000000000000000000000000.0</kp>
+<kd>1000000000000000000000000000.0</kd>
+<mu1>0.1</mu1>
+<mu2>0.1</mu2>
+<material>Gazebo/Yellow</material>
+</gazebo>
     <!-- Plug-ins-->
     <!-- JOINT PUBLISHER -->
     <gazebo>
-        <plugin name="barista_bot_joint_state" filename="libgazebo_ros_joint_state_publisher.so">
+        <plugin name="${robot_name}_bot_joint_state" filename="libgazebo_ros_joint_state_publisher.so">
         <ros>
             <namespace>/${robot_name}</namespace>

File: xacro/cup_holder_tray.xacro (robot description, xacro)
@@ -5,5 +5,5 @@
 <xacro:property name="cup_holder_diameter" value="0.32"/>
 <!-- cup_holder Macro -->
-<xacro:macro name="cup_holder" params="cup_holder_name">
+<xacro:macro name="cup_holder" params="cup_holder_name rviz_material">
   <link name="${cup_holder_name}">
     <visual>
@@ -11,5 +11,5 @@
             <cylinder length="${cup_holder_height}" radius="${cup_holder_diameter/2}"/>
         </geometry>
-        <material name="blue"/>
+        <material name="${rviz_material}"/>
     </visual>
     <collision>
